File: D1-Mini_Adapter.brd (EAGLE design)
At the start: 35 x 42 mm, 26 parts

Commit message: Schaltplan übersichtlicher
Parts:
- RPD: value 4k7 -> 10k
- moved U$2 0.14 mm to (5.00, 37.5)
- renumbered LDR1 to LDR-, LDR2 to LDR+, WEMOS1 to WEMOS
Routing:
- net N$3: track 29.5 -> 24.4 mm
Changed lines of the file:
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@@
 <setting verticaltext="up"/>
 </settings>
-<grid distance="50" unitdist="mil" unit="mil" style="lines" multiple="1" display="yes" altdistance="5" altunitdist="mil" altunit="mil"/>
+<grid distance="2.5" unitdist="mm" unit="mm" style="lines" multiple="1" display="yes" altdistance="5" altunitdist="mil" altunit="mil"/>
 <layers>
 <layer number="1" name="Top" color="4" fill="1" visible="yes" active="yes"/>
@@
 <attribute name="VALUE" x="33.02" y="-0.889" size="0.0254" layer="27"/>
 </element>
-<element name="WEMOS1" library="esp8266modules" package="WEMOS-D1-MINI" value="D1 Mini" x="13.97" y="19.05" smashed="yes">
+<element name="WEMOS" library="esp8266modules" package="WEMOS-D1-MINI" value="D1 Mini" x="13.97" y="19.05" smashed="yes">
 <attribute name="NAME" x="17.13" y="5.27" size="0.6096" layer="25" align="bottom-right"/>
 </element>
@@
 <attribute name="VALUE" x="13.335" y="18.415" size="1.27" layer="27" ratio="10"/>
 </element>
-<element name="U$2" library="holes" library_urn="urn:adsk.eagle:library:237" package="3,3" package3d_urn="urn:adsk.eagle:package:14278/1" value="" x="4.92" y="37.39" smashed="yes"/>
+<element name="U$2" library="holes" library_urn="urn:adsk.eagle:library:237" package="3,3" package3d_urn="urn:adsk.eagle:package:14278/1" value="" x="5" y="37.5" smashed="yes"/>
 <element name="R5" library="resistor" library_urn="urn:adsk.eagle:library:348" package="0207/10" package3d_urn="urn:adsk.eagle:package:23491/2" value="10k" x="15.24" y="22.86" smashed="yes" rot="R180">
 <attribute name="NAME" x="9.525" y="23.495" size="1.27" layer="25" ratio="10"/>
@@
 <attribute name="VALUE" x="10.16" y="39.751" size="0.0254" layer="27"/>
 </element>
-<element name="RPD" library="resistor" library_urn="urn:adsk.eagle:library:348" package="0207/10" package3d_urn="urn:adsk.eagle:package:23491/2" value="4k7" x="15.24" y="34.29" smashed="yes">
+<element name="RPD" library="resistor" library_urn="urn:adsk.eagle:library:348" package="0207/10" package3d_urn="urn:adsk.eagle:package:23491/2" value="10k" x="15.24" y="34.29" smashed="yes">
 <attribute name="NAME" x="9.525" y="34.925" size="1.27" layer="25" ratio="10"/>
 <attribute name="VALUE" x="13.335" y="33.655" size="1.27" layer="27" ratio="10"/>
 </element>
-<element name="LDR1" library="solpad" library_urn="urn:adsk.eagle:library:364" package="SE13" package3d_urn="urn:adsk.eagle:package:26505/1" value="SE13" x="17.78" y="39.37" smashed="yes">
+<element name="LDR-" library="solpad" library_urn="urn:adsk.eagle:library:364" package="SE13" package3d_urn="urn:adsk.eagle:package:26505/1" value="SE13" x="17.78" y="39.37" smashed="yes">
 <attribute name="NAME" x="16.51" y="40.64" size="0.8128" layer="25" ratio="10"/>
 <attribute name="POPULARITY" value="1" x="17.78" y="39.37" size="1.778" layer="27" display="off"/>
 <attribute name="VALUE" x="17.78" y="39.751" size="0.0254" layer="27"/>
 </element>
-<element name="LDR2" library="solpad" library_urn="urn:adsk.eagle:library:364" package="SE13" package3d_urn="urn:adsk.eagle:package:26505/1" value="SE13" x="21.59" y="39.37" smashed="yes">
+<element name="LDR+" library="solpad" library_urn="urn:adsk.eagle:library:364" package="SE13" package3d_urn="urn:adsk.eagle:package:26505/1" value="SE13" x="21.59" y="39.37" smashed="yes">
 <attribute name="NAME" x="20.32" y="40.64" size="0.8128" layer="25" ratio="10"/>
 <attribute name="POPULARITY" value="1" x="21.59" y="39.37" size="1.778" layer="27" display="off"/>
@@
 <signals>
 <signal name="N$12">
-<contactref element="WEMOS1" pad="D6"/>
+<contactref element="WEMOS" pad="D6"/>
 <contactref element="R3" pad="1"/>
 <contactref element="DQ" pad="MP"/>
@@
 <wire x1="10.16" y1="11.43" x2="10.16" y2="12.7" width="0.254" layer="16"/>
 <wire x1="10.16" y1="12.7" x2="1.27" y2="12.7" width="0.254" layer="16"/>
-<contactref element="WEMOS1" pad="D5"/>
+<contactref element="WEMOS" pad="D5"/>
 <wire x1="1.27" y1="12.7" x2="1.27" y2="15.24" width="0.254" layer="16"/>
 <wire x1="1.27" y1="15.24" x2="1.27" y2="17.78" width="0.254" layer="16"/>
@@
 <signal name="GND">
 <contactref element="R1" pad="1"/>
-<contactref element="WEMOS1" pad="GND"/>
+<contactref element="WEMOS" pad="GND"/>
 <contactref element="GND2" pad="MP"/>
 <contactref element="GND" pad="MP"/>
@@
 <signal name="SDA">
 <contactref element="R4" pad="1"/>
-<contactref element="WEMOS1" pad="D2"/>
+<contactref element="WEMOS" pad="D2"/>
 <contactref element="SDA" pad="MP"/>
 <wire x1="20.32" y1="19.05" x2="26.67" y2="19.05" width="1.27" layer="16"/>
@@
 </signal>
 <signal name="+5V">
-<contactref element="WEMOS1" pad="5V"/>
+<contactref element="WEMOS" pad="5V"/>
 <contactref element="+5V" pad="MP"/>
 <contactref element="C2" pad="1"/>
@@
 <wire x1="15.24" y1="19.05" x2="19.05" y2="15.24" width="1.27" layer="16"/>
 <wire x1="19.05" y1="15.24" x2="20.32" y2="15.24" width="1.27" layer="16"/>
-<contactref element="WEMOS1" pad="3V3"/>
+<contactref element="WEMOS" pad="3V3"/>
 <wire x1="3.81" y1="8.89" x2="6.35" y2="8.89" width="1.27" layer="1"/>
 <wire x1="5.08" y1="8.89" x2="3.81" y2="8.89" width="1.27" layer="16"/>
@@
 <wire x1="18.415" y1="24.765" x2="12.065" y2="24.765" width="1.27" layer="16"/>
 <wire x1="12.065" y1="24.765" x2="10.16" y2="22.86" width="1.27" layer="16"/>
-<contactref element="LDR2" pad="MP"/>
+<contactref element="LDR+" pad="MP"/>
 <wire x1="21.59" y1="39.37" x2="24.13" y2="39.37" width="1.27" layer="16"/>
 <wire x1="20.32" y1="30.48" x2="20.32" y2="26.67" width="1.27" layer="16"/>
@@
 </signal>
 <signal name="SCL">
-<contactref element="WEMOS1" pad="D1"/>
+<contactref element="WEMOS" pad="D1"/>
 <contactref element="SCL" pad="MP"/>
 <wire x1="24.13" y1="21.59" x2="26.67" y2="21.59" width="1.27" layer="16"/>
@@
 </signal>
 <signal name="N$3">
-<contactref element="LDR1" pad="MP"/>
 <contactref element="RPD" pad="2"/>
-<contactref element="WEMOS1" pad="A0"/>
+<contactref element="WEMOS" pad="A0"/>
 <wire x1="6.985" y1="32.385" x2="6.35" y2="31.75" width="1.27" layer="1"/>
 <wire x1="15.875" y1="32.385" x2="17.78" y2="34.29" width="1.27" layer="1"/>
@@
 <wire x1="5.08" y1="24.13" x2="6.35" y2="25.4" width="1.27" layer="1"/>
 <wire x1="5.08" y1="24.13" x2="3.81" y2="24.13" width="1.27" layer="1"/>
-<wire x1="17.78" y1="34.29" x2="17.78" y2="39.37" width="1.27" layer="1"/>
+<contactref element="LDR-" pad="MP"/>
+<wire x1="20.32" y1="34.29" x2="17.78" y2="39.37" width="0" layer="19" extent="1-1"/>
 </signal>
 </signals>
