File: D1-Mini_Adapter_V4.brd (EAGLE design)
At the start: 35 x 42 mm, 26 parts

Commit message: New PCS Version 4.1
Parts:
- removed RES2: SE13, solpad:SE13
- added GN, SC, SD, SW0: SE13, solpad:SE13
- added VIN: LSP13, solpad:LSP13
- moved RES1 3.81 mm to (10.2, 39.4), turned to 0 degrees
- moved U$2 0.50 mm to (5.00, 37.0)
Connections:
- net N$12 renamed DQ
- net N$20 renamed D5
- net N$22 renamed REST
- removed net N$4: R6.1, RES1.MP
- new net SW0: R6.1, SW0.MP, WEMOS.D7
- net 3V3: now also VIN.MP
- net GND: now also GN.MP
- net N$5: now also RES1.MP; no longer RES2.MP
- net SCL: now also SC.MP
- net SDA: now also SD.MP
Routing:
- net SW0: track 0.00 -> 32.9 mm
- net N$4: track 16.8 -> 0.00 mm
- net D5: track 22.1 -> 30.9 mm
- net N$3: track 24.4 -> 29.5 mm
- net REST: track 13.8 -> 18.3 mm
- net 3V3: track 80.8 -> 78.2 mm
- net +5V: track 14.2 -> 16.3 mm
Other:
- board text added: "(C) Michael Hufschmidt, Sept. 2023"
- board text added: "D1-Mini Adapter V4.1"
- board text removed: "(C) Michael Hufschmidt, Dez. 2022"
- board text removed: "D1-Mini Adapter V3.2"

Commit message: PCB and schema Version 4.2
Parts:
- moved RES1 3.81 mm to (14.0, 39.4)
- moved SW0 3.81 mm to (10.2, 39.4), turned to 180 degrees
Connections:
- net N$3 renamed LDR
- net N$5 renamed RES1
Routing:
- net SW0: track 32.9 -> 36.5 mm, vias 0 -> 1
- net RES1: track 11.0 -> 10.5 mm
- net GND: vias 2 -> 3
Other:
- board text added: "(C) Michael Hufschmidt, Okt. 2023"
- board text added: "D1-Mini Adapter V4.2"
- board text removed: "(C) Michael Hufschmidt, Sept. 2023"
- board text removed: "D1-Mini Adapter V4.1"
Changed lines of the file:
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@@
 <setting verticaltext="up"/>
 </settings>
-<grid distance="25" unitdist="mil" unit="mil" style="lines" multiple="1" display="yes" altdistance="5" altunitdist="mil" altunit="mil"/>
+<grid distance="12.5" unitdist="mil" unit="mil" style="lines" multiple="1" display="yes" altdistance="5" altunitdist="mil" altunit="mil"/>
 <layers>
 <layer number="1" name="Top" color="4" fill="1" visible="yes" active="yes"/>
@@
 <board>
 <plain>
-<text x="1.905" y="10.335" size="1.27" layer="21" rot="R90">D1-Mini Adapter V4.1</text>
+<text x="1.905" y="10.335" size="1.27" layer="21" rot="R90">D1-Mini Adapter V4.2</text>
 <text x="30.48" y="2.54" size="0.8128" layer="21" rot="R90">---- IKEA ----</text>
 <text x="30.48" y="22.86" size="0.8128" layer="21" rot="R90">Ext. 1 Wire</text>
@@
 <wire x1="0" y1="42" x2="35" y2="42" width="0.127" layer="20"/>
 <wire x1="0" y1="42" x2="0" y2="0" width="0.127" layer="20"/>
-<text x="8.255" y="10.795" size="0.8128" layer="21" rot="R90">(C) Michael Hufschmidt, Sept. 2023</text>
+<text x="8.255" y="10.795" size="0.8128" layer="21" rot="R90">(C) Michael Hufschmidt, Okt. 2023</text>
 </plain>
 <attributes>
@@
 <attribute name="VALUE" x="13.335" y="29.845" size="1.27" layer="27" ratio="10"/>
 </element>
-<element name="SW0" library="solpad" library_urn="urn:adsk.eagle:library:364" package="SE13" package3d_urn="urn:adsk.eagle:package:26505/1" value="SE13" x="13.97" y="39.37" smashed="yes" rot="R90">
+<element name="SW0" library="solpad" library_urn="urn:adsk.eagle:library:364" package="SE13" package3d_urn="urn:adsk.eagle:package:26505/1" value="SE13" x="10.16" y="39.37" smashed="yes" rot="R180">
+<attribute name="NAME" x="8.9535" y="40.64" size="0.8128" layer="25" ratio="10"/>
+<attribute name="POPULARITY" value="1" x="10.16" y="39.37" size="1.778" layer="27" rot="R180" display="off"/>
+<attribute name="VALUE" x="10.16" y="38.989" size="0.0254" layer="27" rot="R180"/>
+</element>
+<element name="RES1" library="solpad" library_urn="urn:adsk.eagle:library:364" package="SE13" package3d_urn="urn:adsk.eagle:package:26505/1" value="SE13" x="13.97" y="39.37" smashed="yes">
 <attribute name="NAME" x="12.7" y="40.64" size="0.8128" layer="25" ratio="10"/>
-<attribute name="POPULARITY" value="1" x="13.97" y="39.37" size="1.778" layer="27" rot="R90" display="off"/>
-<attribute name="VALUE" x="13.589" y="39.37" size="0.0254" layer="27" rot="R90"/>
-</element>
-<element name="RES1" library="solpad" library_urn="urn:adsk.eagle:library:364" package="SE13" package3d_urn="urn:adsk.eagle:package:26505/1" value="SE13" x="10.16" y="39.37" smashed="yes">
-<attribute name="NAME" x="8.89" y="40.64" size="0.8128" layer="25" ratio="10"/>
-<attribute name="POPULARITY" value="1" x="10.16" y="39.37" size="1.778" layer="27" display="off"/>
-<attribute name="VALUE" x="10.16" y="39.751" size="0.0254" layer="27"/>
+<attribute name="POPULARITY" value="1" x="13.97" y="39.37" size="1.778" layer="27" display="off"/>
+<attribute name="VALUE" x="13.97" y="39.751" size="0.0254" layer="27"/>
 </element>
 <element name="RPD" library="resistor" library_urn="urn:adsk.eagle:library:348" package="0207/10" package3d_urn="urn:adsk.eagle:package:23491/2" value="10k" x="15.24" y="34.29" smashed="yes">
@@
 <wire x1="33.02" y1="16.51" x2="39.37" y2="8.89" width="0" layer="19" extent="1-1"/>
 </signal>
-<signal name="N$5">
+<signal name="RES1">
 <contactref element="R7" pad="1"/>
 <contactref element="RES1" pad="MP"/>
-<wire x1="10.16" y1="39.37" x2="12.7" y2="36.83" width="1.27" layer="16"/>
-<wire x1="12.7" y1="36.83" x2="12.7" y2="33.02" width="1.27" layer="16"/>
-<wire x1="12.7" y1="33.02" x2="10.16" y2="30.48" width="1.27" layer="16"/>
-</signal>
-<signal name="N$3">
+<wire x1="13.97" y1="39.37" x2="13.97" y2="34.29" width="0.8128" layer="16"/>
+<wire x1="13.97" y1="34.29" x2="10.16" y2="30.48" width="1.27" layer="16"/>
+</signal>
+<signal name="LDR">
 <contactref element="RPD" pad="2"/>
 <contactref element="WEMOS" pad="A0"/>
@@
 <contactref element="R6" pad="1"/>
 <contactref element="SW0" pad="MP"/>
-<wire x1="15.24" y1="30.48" x2="11.43" y2="26.67" width="1.27" layer="16"/>
+<wire x1="11.43" y1="26.67" x2="15.875" y2="31.115" width="0.8128" layer="16"/>
 <wire x1="11.43" y1="26.67" x2="10.16" y2="26.67" width="1.27" layer="16"/>
-<wire x1="13.97" y1="39.37" x2="15.24" y2="38.1" width="1.27" layer="16"/>
-<wire x1="15.24" y1="30.48" x2="15.24" y2="38.1" width="1.27" layer="16"/>
 <wire x1="10.16" y1="26.67" x2="7.62" y2="24.13" width="1" layer="16"/>
 <wire x1="7.62" y1="24.13" x2="7.62" y2="15.91980625" width="0.5" layer="16"/>
@@
 <wire x1="6.35" y1="14.64980625" x2="6.35" y2="13.97" width="0.508" layer="16"/>
 <wire x1="3.81" y1="13.97" x2="6.35" y2="13.97" width="0.508" layer="16"/>
+<wire x1="15.875" y1="31.115" x2="15.875" y2="36.195" width="0.8128" layer="16"/>
+<via x="15.875" y="36.195" extent="1-16" drill="0.35"/>
+<wire x1="15.875" y1="36.195" x2="13.335" y2="36.195" width="0.8128" layer="1"/>
+<wire x1="13.335" y1="36.195" x2="10.16" y2="39.37" width="0.8128" layer="1"/>
 </signal>
 <signal name="GND">
@@
 <wire x1="30.48" y1="28.575" x2="30.48" y2="22.86" width="1.27" layer="16"/>
 <wire x1="31.75" y1="40.64" x2="30.48" y2="39.37" width="1.27" layer="16"/>
-<wire x1="10.16" y1="34.29" x2="8.255" y2="32.385" width="1.27" layer="16"/>
-<wire x1="8.255" y1="32.385" x2="8.255" y2="29.21" width="1.27" layer="16"/>
 <via x="8.255" y="29.21" extent="1-16" drill="0.35"/>
 <wire x1="8.255" y1="29.21" x2="8.89" y2="28.575" width="0.8128" layer="1"/>
@@
 <wire x1="33.3502" y1="40.64" x2="31.75" y2="40.64" width="1.27" layer="16"/>
 <wire x1="29.21" y1="39.37" x2="30.48" y2="39.37" width="1.27" layer="16"/>
+<via x="8.255" y="29.21" extent="1-16" drill="0.35"/>
+<wire x1="8.255" y1="29.21" x2="8.255" y2="32.385" width="0.8128" layer="16"/>
+<wire x1="8.255" y1="32.385" x2="10.16" y2="34.29" width="0.8128" layer="16"/>
 <wire x1="33.02" y1="20.32" x2="39.37" y2="13.97" width="0" layer="19" extent="1-1"/>
 </signal>
